File: hardware/motherboard/irq_handler.kicad_sch (KiCad schematic)
At the start: 16 parts, among them U14 74HCT02, U17 74HCT148, U18 74HCT148, U23 74HCT00, U24 74HCT85, U25 74HCT574, U26 74HCT574

Commit message: A lot of updates
Changed lines of the file:
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@@
 	(wire
 		(pts
-			(xy 115.57 156.21) (xy 115.57 127)
+			(xy 120.65 127) (xy 120.65 156.21)
 		)
 		(stroke
@@
 	(wire
 		(pts
-			(xy 114.3 118.11) (xy 116.84 118.11)
-		)
-		(stroke
-			(width 0)
-			(type default)
-		)
-	)
-	(wire
-		(pts
-			(xy 113.03 156.21) (xy 115.57 156.21)
+			(xy 113.03 156.21) (xy 120.65 156.21)
 		)
 		(stroke
@@
 	(wire
 		(pts
+			(xy 116.84 81.28) (xy 128.27 81.28)
+		)
+		(stroke
+			(width 0)
+			(type default)
+		)
+	)
+	(wire
+		(pts
 			(xy 33.02 110.49) (xy 41.91 110.49)
 		)
@@
 	(wire
 		(pts
-			(xy 114.3 139.7) (xy 114.3 118.11)
+			(xy 116.84 81.28) (xy 116.84 139.7)
 		)
 		(stroke
@@
 	(wire
 		(pts
-			(xy 87.63 139.7) (xy 114.3 139.7)
+			(xy 87.63 139.7) (xy 116.84 139.7)
 		)
 		(stroke
@@
 	(wire
 		(pts
-			(xy 116.84 124.46) (xy 119.38 124.46)
-		)
-		(stroke
-			(width 0)
-			(type default)
-		)
-	)
-	(wire
-		(pts
 			(xy 113.03 87.63) (xy 113.03 114.3)
 		)
@@
 	(wire
 		(pts
-			(xy 121.92 143.51) (xy 121.92 129.54)
+			(xy 121.92 129.54) (xy 121.92 153.67)
 		)
 		(stroke
@@
 	(wire
 		(pts
-			(xy 116.84 81.28) (xy 128.27 81.28)
-		)
-		(stroke
-			(width 0)
-			(type default)
-		)
-	)
-	(wire
-		(pts
-			(xy 116.84 81.28) (xy 116.84 118.11)
-		)
-		(stroke
-			(width 0)
-			(type default)
-		)
-	)
-	(wire
-		(pts
 			(xy 119.38 124.46) (xy 128.27 124.46)
 		)
@@
 	(wire
 		(pts
-			(xy 113.03 158.75) (xy 116.84 158.75)
+			(xy 113.03 158.75) (xy 119.38 158.75)
 		)
 		(stroke
@@
 	(wire
 		(pts
-			(xy 116.84 158.75) (xy 116.84 124.46)
+			(xy 119.38 158.75) (xy 119.38 124.46)
 		)
 		(stroke
@@
 	(wire
 		(pts
-			(xy 114.3 153.67) (xy 114.3 143.51)
-		)
-		(stroke
-			(width 0)
-			(type default)
-		)
-	)
-	(wire
-		(pts
 			(xy 153.67 111.76) (xy 156.21 111.76)
 		)
@@
 	(wire
 		(pts
-			(xy 114.3 143.51) (xy 121.92 143.51)
-		)
-		(stroke
-			(width 0)
-			(type default)
-		)
-	)
-	(wire
-		(pts
 			(xy 113.03 161.29) (xy 118.11 161.29)
 		)
@@
 	(wire
 		(pts
-			(xy 115.57 127) (xy 120.65 127)
-		)
-		(stroke
-			(width 0)
-			(type default)
-		)
-	)
-	(wire
-		(pts
-			(xy 118.11 121.92) (xy 118.11 73.66)
+			(xy 118.11 73.66) (xy 118.11 121.92)
 		)
 		(stroke
@@
 	(wire
 		(pts
-			(xy 113.03 153.67) (xy 114.3 153.67)
-		)
-		(stroke
+			(xy 113.03 153.67) (xy 121.92 153.67)
+		)
+		(stroke
