File: hardware/motherboard/ps2.kicad_sch (KiCad schematic)
At the start: 26 parts, among them J1 Mouse, J2 Keyboard, U10 74HCT573, U11 74HCT595, U12 74HCT595, U13 74HCT573, U5 74HCT32, U6 74HCT14, U7 74HCT595, U8 74HCT595, U9 74HCT14

Commit message: A lot of updates
Parts:
- removed J1: Mouse, motherboard:mini-DIN 6, symbol Connector:Mini-DIN-6
- removed J2: Keyboard, motherboard:mini-DIN 6, symbol Connector:Mini-DIN-6
- added J7: ~, kicad-lib:2xPS2-Mini-Din, symbol motherboard:2xPS2
Connections:
- net GND: now also J7.3 (Mouse_GND), J7.9 (Kbd_GND), J7.G (GND); no longer C18.2, C19.2
- net PS2_KB_CLK: now also J7.11 (Kbd_Clock)
- net PS2_KB_DATA: now also J7.7 (Kbd_Data)
- net PS2_M_CLK: now also J7.5 (Mouse_Clock)
- net PS2_M_DATA: now also J7.1 (Mouse_Data)
- net VCC: now also J7.10 (Kbd_PWR), J7.4 (Mouse_PWR); no longer C18.1, C19.1
- no-connect marks 22 -> 18
Other:
- moved on the sheet: C18, C19
