File: hardware/motherboard/serial.kicad_sch (KiCad schematic)
At the start: 25 parts, among them J3 Serial, J4 Console, J7 LCD, Q1 NPN, U15 MCP2221A, U28 6522, U30 MAX232, U31 68C681, Y1 Crystal

Commit message: A lot of updates
Parts:
- removed C30: 10u, Capacitor_THT:CP_Radial_D4.0mm_P2.00mm, symbol Device:C_Polarized
- removed J7: LCD, Connector_PinHeader_2.54mm:PinHeader_2x08_P2.54mm_Vertical, symbol Connector_Generic:Conn_02x08_Odd_Even
- removed Q1: NPN, Package_TO_SOT_THT:TO-92L_Inline, symbol Device:Q_NPN_ECB
- removed R6: 220, Resistor_THT:R_Axial_DIN0204_L3.6mm_D1.6mm_P7.62mm_Horizontal, symbol Device:R
- removed R7: 1k, Resistor_THT:R_Axial_DIN0204_L3.6mm_D1.6mm_P7.62mm_Horizontal, symbol Device:R
- removed RV1: 10k, Potentiometer_THT:Potentiometer_Vishay_T73YP_Vertical, symbol Device:R_Potentiometer
Connections:
- no-connect marks 41 -> 37
